Commit message: Update lidars

File: sam_bot_description/src/description/sam_bot_description.urdf (robot description, URDF)
Before this commit: robot sam_bot, 6 links, 5 joints
Links:
- removed link lidar_link
- added link lidar1_link, mass 0.125; collision cylinder length=0.055 radius=0.0508; visual cylinder length=0.055 radius=0.0508
- added link lidar2_link, mass 0.125; collision cylinder length=0.055 radius=0.0508; visual cylinder length=0.055 radius=0.0508
Joints:
- removed joint lidar_joint
- added joint lidar1_joint: type fixed, parent base_link, child lidar1_link, origin xyz=0.75 -0.45 0.12 rpy=0 0 0
- added joint lidar2_joint: type fixed, parent base_link, child lidar2_link, origin xyz=-0.75 0.45 0.12 rpy=0 0 0
